File: pcb/v2-kicad5/pa3gyf-gpsdocxo-2016-v2/pa3gyf-gpsdocxo-2016-v2-ocxo-r1.sch (KiCad schematic (older format))
At the start: 0 parts

Commit message: Committing apparent changes in working directory.
Parts:
- added C302, C303, C311: 1u, Capacitors_SMD:C_0805_HandSoldering, symbol pa3gyf-gpsdocxo-2016-v2-rescue:C_Small-pa3gyf-gpsdocxo-2016-ocxo-r1-cache-saved
- added C304, C305: 10u, Resistors_SMD:R_0805_HandSoldering, symbol pa3gyf-gpsdocxo-2016-v2-rescue:CP_Small-pa3gyf-gpsdocxo-2016-ocxo-r1-cache-saved
- added C306, C307, C308, C309: 1n, Capacitors_SMD:C_0805_HandSoldering, symbol pa3gyf-gpsdocxo-2016-v2-rescue:C_Small-pa3gyf-gpsdocxo-2016-ocxo-r1-cache-saved
- added C310: 100u, Capacitors_Elko_ThroughHole:Elko_vert_11.5x8mm_RM3.5, symbol pa3gyf-gpsdocxo-2016-v2-rescue:CP_Small-pa3gyf-gpsdocxo-2016-ocxo-r1-cache-saved
- added L301, L302: 22uH, Capacitors_SMD:C_0805_HandSoldering, symbol pa3gyf-gpsdocxo-2016-v2-rescue:L_Small-pa3gyf-gpsdocxo-2016-ocxo-r1-cache-saved
- added R301: 2R/5W, Resistors_ThroughHole:Resistor_Ceramic_Horizontal_L23mm-W9mm-H9mm-p30mm, symbol pa3gyf-gpsdocxo-2016-v2-rescue:R-pa3gyf-gpsdocxo-2016-ocxo-r1-cache-saved
- added R302, R304, R305, R306, R309, R310: InfR, Resistors_SMD:R_0805_HandSoldering, symbol pa3gyf-gpsdocxo-2016-v2-rescue:R-pa3gyf-gpsdocxo-2016-ocxo-r1-cache-saved
- added R303, R307, R308: 0R, Resistors_SMD:R_0805_HandSoldering, symbol pa3gyf-gpsdocxo-2016-v2-rescue:R-pa3gyf-gpsdocxo-2016-ocxo-r1-cache-saved
- added U301: 78S12, Transistors_TO-220:TO-220_Neutral123_Vertical_LargePads, symbol pa3gyf-gpsdocxo-2016-v2-rescue:LM7812-pa3gyf-gpsdocxo-2016-ocxo-r1-cache-saved
- added U302: MV89, MORION_FULLMETA:MV89, symbol pa3gyf-gpsdocxo-2016-v2-rescue:MV89-pa3gyf-gpsdocxo-2016-ocxo-r1-cache-saved
- added U303: ADP-2-1, MiniCircuits:CD636, symbol pa3gyf-gpsdocxo-2016-v2-rescue:ADP-2-1+-pa3gyf-gpsdocxo-2016-ocxo-r1-cache-saved
Connections:
- new net: R302.1, R303.2, U302.3 (RF)
- new net: R303.1, R304.1, U303.1 (IN)
- new net: R306.1, R308.2, U303.4 (OUT2)
- new net: R305.1, R307.2, U303.3 (OUT1)
- new net: C309.1, L302.2, U302.1 (Uin)
- new net: C308.1, L301.2, U302.2 (Uref)
- new net: C310.1, C311.1, U301.VO, U302.5 (Us)
- new net: U303.2 (CON1), U303.5 (CON2)
- new net 10MHz_out_1: R307.1, R309.1
- new net 10MHz_out_2: R308.1, R310.1
- new net GND: C302.2, C303.2, C304.2, C305.2, C306.2, C307.2, C308.2, C309.2, C310.2, C311.2, R302.2, R304.2, R305.2, R306.2, R309.2, R310.2, U301.GND, U302.4 (GND), U303.6 (GND)
- new net V21u: C303.1, R301.1
- new net Vref: C304.1, C306.1, L301.1
- new net Vsense: C302.1, R301.2, U301.VI
- new net Vtune: C305.1, C307.1, L302.1
Other:
- note added: "-3.13 dB"
- note added: "ISO >= 34.5 dB @ 10 MHz"
- note added: "OCXO Ouput\nSplitter/Isolator"
- note added: "OCXO Output\nMatching"
- note added: "OCXO PLL Interface"
- note added: "OCXO Power Supply\nand Current Sense"
